Commit message: need to fix collision

File: models/drake/iiwa_description/urdf/iiwa14_polytope_collision.urdf (robot description, URDF)
Before this commit: robot iiwa14, 11 links, 10 joints
Links:
- link iiwa_link_1: geometry collision cylinder length=0.29 radius=0.101; visual mesh filename=../meshes/visual/link_1.obj
- link iiwa_link_2: geometry collision cylinder length=0.29 radius=0.101; visual mesh filename=../meshes/visual/link_2.obj
- link iiwa_link_3: geometry collision cylinder length=0.29 radius=0.092; visual mesh filename=../meshes/visual/link_3.obj
- link iiwa_link_4: geometry collision cylinder length=0.25 radius=0.092; visual mesh filename=../meshes/visual/link_4.obj

File: models/drake/iiwa_description/urdf/iiwa14_primitive_collision.urdf (robot description, URDF)
Before this commit: robot iiwa14, 11 links, 10 joints
Links:
- link iiwa_link_0: geometry collision mesh filename=../meshes/visual/link_0.obj
- link iiwa_link_1: geometry collision mesh filename=../meshes/visual/link_1.obj; visual cylinder length=0.29 radius=0.101
- link iiwa_link_2: geometry collision mesh filename=../meshes/visual/link_2.obj; visual cylinder length=0.29 radius=0.101
- link iiwa_link_3: geometry collision mesh filename=../meshes/visual/link_3.obj; visual cylinder length=0.29 radius=0.092
- link iiwa_link_4: geometry collision mesh filename=../meshes/visual/link_4.obj; visual cylinder length=0.25 radius=0.092
- link iiwa_link_5: geometry collision mesh filename=../meshes/visual/link_5.obj; visual cylinder length=0.29 radius=0.07
- link iiwa_link_6: geometry collision mesh filename=../meshes/visual/link_6.obj; visual mesh filename=../meshes/collision/link_6.obj
- link iiwa_link_7: geometry collision mesh filename=../meshes/visual/link_7.obj; visual mesh filename=../meshes/collision/link_7.obj

File: models/stove.urdf (robot description, URDF)
Before this commit: robot stove, 1 links, 0 joints
Links:
- link base_link: geometry collision box size=0.2499 0.2499 0.0499; collision sphere radius=1e-7

Commit message: sync

File: models/drake/iiwa_description/urdf/iiwa14_polytope_collision.urdf (robot description, URDF)
Before this commit: robot iiwa14, 11 links, 10 joints
Links:
- link iiwa_link_5: geometry collision cylinder length=0.29 radius=0.07; visual mesh filename=../meshes/visual/link_5.obj
